File: balancer.kicad_pcb (KiCad board)
At the start: 2 copper layers, 71.1 x 52.6 mm, 19 parts, among them J3 AVR-ISP-6, J4 Screw_Terminal_01x03, Q1 IRLZ34N, U1 EL817, U2 ATtiny85-20PU

Commit message: changed VBATT connector from 2 GND to 2 VBATT
Parts:
- moved C3 180.2 mm to (132.6, 113.5)
- moved D1 180.2 mm to (164.3, 91.9)
- moved R1 180.2 mm to (164.3, 94.7)
- moved TX1 180.2 mm to (165.9, 113.3)
- moved C2 180.2 mm to (145.0, 105.2)
- moved J3 180.2 mm to (144.3, 120.4)
- moved J4 180.2 mm to (105.9, 121.9)
- moved R2 180.2 mm to (102.1, 80.0)
- moved R3 180.2 mm to (102.1, 94.0)
- moved R4 180.2 mm to (126.2, 119.1)
- moved R6 180.2 mm to (149.9, 120.7)
- moved U2 180.2 mm to (137.7, 109.2)
- moved C1 180.2 mm to (153.2, 109.2)
- moved D2 180.2 mm to (130.6, 119.1)
- moved Q1 180.2 mm to (168.1, 82.5)
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Connections:
- J4 pad 2: GND -> +BATT
Routing:
- net +BATT: track 99.5 -> 124.1 mm
